File: pcb/crn-x-kbd-choc.kicad_sch (KiCad schematic)
At the start: 49 parts, among them SW1 SW_PUSH, SW10 SW_PUSH, SW11 SW_PUSH, SW12 SW_PUSH, SW13 SW_PUSH, SW14 SW_PUSH, SW15 SW_PUSH, SW16 SW_PUSH, SW17 SW_PUSH, SW18 SW_PUSH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

Commit message: doc
Other:
- note added: "POWER SWITCH 1"
- note added: "POWER SWITCH 2"
- note removed: "P O W E R S W I T C H"
- moved on the sheet: PWR_2
